Commit message: add mass intertis

File: chapt6/chapt6_ws/src/fishbot_description/urdf/fishbot/actuator/caster.urdf.xacro (robot description, xacro)
@@ -2,42 +2,39 @@
 <robot xmlns:xacro="http://www.ros.org/wiki/xacro">
     <xacro:include filename="$(find fishbot_description)/urdf/fishbot/common_intertia.urdf.xacro"/>
-    <xacro:macro name="imu_xacro" params="xyz">
+    <xacro:macro name="caster_xacro" params="caster_name xyz">
         <!-- 机器人的惯性测量单元 -->
-        <link name="imu_link">
+        <link name="${caster_name}_link">
             <!-- 部件的外观描述 -->
             <visual>
-                <!-- 沿着自身几何中心的偏移量和旋转量 -->
-                <origin xyz="0.0 0.0 0.0" rpy="0.0 0.0 0.0"/>
-                <!-- 几何形状 -->
+                <origin xyz="0.0 0.0 0.0" rpy="1.57079 0.0 0.0"/>
                 <geometry>
-                    <box size="0.02 0.02 0.02"/>
+                    <sphere radius="0.016"/>
                 </geometry>
                 <!-- 材质 颜色 -->
-                <material name="black">
-                    <color rgba="0.0 0.0 0.0 0.5"/>
+                <material name="yellow">
+                    <color rgba="1.0 1.0 0.0 1.0"/>
                 </material>
             </visual>
             <collision>
-                <!-- 沿着自身几何中心的偏移量和旋转量 -->
-                <origin xyz="0.0 0.0 0.0" rpy="0.0 0.0 0.0"/>
-                <!-- 几何形状 -->
+                <origin xyz="0.0 0.0 0.0" rpy="1.57079 0.0 0.0"/>
                 <geometry>
-                    <box size="0.02 0.02 0.02"/>
+                    <sphere radius="0.016"/>
                 </geometry>
                 <!-- 材质 颜色 -->
-                <material name="black">
-                    <color rgba="0.0 0.0 0.0 0.5"/>
+                <material name="yellow">
+                    <color rgba="1.0 1.0 0.0 1.0"/>
                 </material>
             </collision>
-            <xacro:box_intertia m="0.2" w="0.02" h="0.02" d="0.02"/>
+            <xacro:sphere_intertia m="0.2" r="0.016"/>
         </link>
         <!-- 机器人的关节 用于组合机器人的部件-->
-        <joint name="imu_joint" type="fixed">
+        <joint name="${caster_name}_joint" type="fixed">
             <!-- 关节的父部件 -->
             <parent link="base_link"/>
             <!-- 关节的子部件 -->
-            <child link="imu_link"/>
+            <child link="${caster_name}_link"/>
             <!-- 关节的位置和旋转 -->
             <origin xyz="${xyz}" rpy="0.0 0.0 0.0"/>
+            <axis xyz="0 1 0"/>
         </joint>
     </xacro:macro>

File: chapt6/chapt6_ws/src/fishbot_description/urdf/fishbot/actuator/wheel.urdf.xacro (robot description, xacro)
@@ -2,42 +2,39 @@
 <robot xmlns:xacro="http://www.ros.org/wiki/xacro">
     <xacro:include filename="$(find fishbot_description)/urdf/fishbot/common_intertia.urdf.xacro"/>
-    <xacro:macro name="imu_xacro" params="xyz">
+    <xacro:macro name="wheel_xacro" params="wheel_name xyz">
         <!-- 机器人的惯性测量单元 -->
-        <link name="imu_link">
+        <link name="${wheel_name}_link">
             <!-- 部件的外观描述 -->
             <visual>
-                <!-- 沿着自身几何中心的偏移量和旋转量 -->
-                <origin xyz="0.0 0.0 0.0" rpy="0.0 0.0 0.0"/>
-                <!-- 几何形状 -->
+                <origin xyz="0.0 0.0 0.0" rpy="1.57079 0.0 0.0"/>
                 <geometry>
-                    <box size="0.02 0.02 0.02"/>
+                    <cylinder radius="0.032" length="0.04"/>
                 </geometry>
                 <!-- 材质 颜色 -->
-                <material name="black">
-                    <color rgba="0.0 0.0 0.0 0.5"/>
+                <material name="yellow">
+                    <color rgba="1.0 1.0 0.0 1.0"/>
                 </material>
             </visual>
             <collision>
-                <!-- 沿着自身几何中心的偏移量和旋转量 -->
-                <origin xyz="0.0 0.0 0.0" rpy="0.0 0.0 0.0"/>
-                <!-- 几何形状 -->
+                <origin xyz="0.0 0.0 0.0" rpy="1.57079 0.0 0.0"/>
                 <geometry>
-                    <box size="0.02 0.02 0.02"/>
+                    <cylinder radius="0.032" length="0.04"/>
                 </geometry>
                 <!-- 材质 颜色 -->
-                <material name="black">
-                    <color rgba="0.0 0.0 0.0 0.5"/>
+                <material name="yellow">
+                    <color rgba="1.0 1.0 0.0 1.0"/>
                 </material>
             </collision>
-            <xacro:box_intertia m="0.2" w="0.02" h="0.02" d="0.02"/>
+            <xacro:cylinder_intertia m="0.5" r="0.032" h="0.04"/>
         </link>
         <!-- 机器人的关节 用于组合机器人的部件-->
-        <joint name="imu_joint" type="fixed">
+        <joint name="${wheel_name}_joint" type="continuous">
             <!-- 关节的父部件 -->
             <parent link="base_link"/>
             <!-- 关节的子部件 -->
-            <child link="imu_link"/>
+            <child link="${wheel_name}_link"/>
             <!-- 关节的位置和旋转 -->
             <origin xyz="${xyz}" rpy="0.0 0.0 0.0"/>
+            <axis xyz="0 1 0"/>
         </joint>
     </xacro:macro>

File: chapt6/chapt6_ws/src/fishbot_description/urdf/fishbot/base.urdf.xacro (robot description, xacro)
@@ -1,5 +1,7 @@
 <?xml version="1.0"?>
 <robot xmlns:xacro="http://www.ros.org/wiki/xacro">
+    <xacro:include filename="$(find fishbot_description)/urdf/fishbot/common_intertia.urdf.xacro"/>
     <xacro:macro name="base_xacro" params="length radius">
+        <link name="base_footPrint"/>
         <!-- 机器人的身体部分 -->
         <link name="base_link">
@@ -18,5 +20,27 @@
                 </material>
             </visual>
+            <collision>
+                <!-- 沿着自身几何中心的偏移量和旋转量 -->
+                <origin xyz="0.0 0.0 0.0" rpy="0.0 0.0 0.0"/>
+                <!-- 几何形状 -->
+                <geometry>
+                    <!-- 圆柱体 -->
+                    <cylinder radius="${radius}" length="${length}"/>
+                </geometry>
+                <!-- 材质 颜色 -->
+                <material name="white">
+                    <color rgba="1.0 1.0 1.0 0.5"/>
+                </material>
+            </collision>
+            <xacro:cylinder_intertia m="1.0" r="${radius}" h="${length}"/>
         </link>
+        <joint name="base_joint" type="fixed">
+            <!-- 关节的父部件 -->
+            <parent link="base_footPrint"/>
+            <!-- 关节的子部件 -->
+            <child link="base_link"/>
+            <!-- 关节的位置和旋转 -->
+            <origin xyz="0.0 0.0 ${length/2+0.032-0.001}" rpy="0.0 0.0 0.0"/>
+        </joint>
     </xacro:macro>
 </robot>

File: chapt6/chapt6_ws/src/fishbot_description/urdf/fishbot/fishbot.urdf.xacro (robot description, xacro)
@@ -1,11 +1,20 @@
 <?xml version="1.0"?>
 <robot xmlns:xacro="http://www.ros.org/wiki/xacro" name="fishbot">
+<!-- 基础部分 -->
 <xacro:include filename="$(find fishbot_description)/urdf/fishbot/base.urdf.xacro"/>
+<!-- 传感器部分 -->
 <xacro:include filename="$(find fishbot_description)/urdf/fishbot/sensor/laser.urdf.xacro"/>
 <xacro:include filename="$(find fishbot_description)/urdf/fishbot/sensor/camera.urdf.xacro"/>
 <xacro:include filename="$(find fishbot_description)/urdf/fishbot/sensor/imu.urdf.xacro"/>
+<!-- 执行器部分 -->
+<xacro:include filename="$(find fishbot_description)/urdf/fishbot/actuator/wheel.urdf.xacro"/>
+<xacro:include filename="$(find fishbot_description)/urdf/fishbot/actuator/caster.urdf.xacro"/>
 <xacro:base_xacro length="0.12" radius="0.1"/>
 <xacro:laser_xacro xyz="0.0 0.0 0.10"/>
 <xacro:camera_xacro xyz="0.10 0.0 0.075"/>
 <xacro:imu_xacro xyz="0.0 0.0 0.02"/>
+<xacro:wheel_xacro wheel_name="left_wheel" xyz="0.0 0.10 -0.06"/>
+<xacro:wheel_xacro wheel_name="right_wheel" xyz="0.0 -0.10 -0.06"/>
+<xacro:caster_xacro caster_name="front_caster" xyz="0.08 0.0 -0.076"/>
+<xacro:caster_xacro caster_name="back_caster" xyz="-0.08 0.0 -0.076"/>
 </robot>

File: chapt6/chapt6_ws/src/fishbot_description/urdf/fishbot/sensor/camera.urdf.xacro (robot description, xacro)
@@ -1,4 +1,5 @@
 <?xml version="1.0"?>
 <robot xmlns:xacro="http://www.ros.org/wiki/xacro">
+    <xacro:include filename="$(find fishbot_description)/urdf/fishbot/common_intertia.urdf.xacro"/>
     <xacro:macro name="camera_xacro" params="xyz">
         <link name="camera_link">
@@ -9,5 +10,4 @@
                 <!-- 几何形状 -->
                 <geometry>
-                    <!-- 正方体 -->
                     <box size="0.02 0.10 0.02"/>
                 </geometry>
@@ -17,4 +17,17 @@
                 </material>
             </visual>
+            <collision>
+                <!-- 沿着自身几何中心的偏移量和旋转量 -->
+                <origin xyz="0.0 0.0 0.0" rpy="0.0 0.0 0.0"/>
+                <!-- 几何形状 -->
+                <geometry>
+                    <box size="0.02 0.10 0.02"/>
+                </geometry>
+                <!-- 材质 颜色 -->
+                <material name="black">
+                    <color rgba="0.0 0.0 0.0 0.5"/>
+                </material>
+            </collision>
+            <xacro:box_intertia m="0.3" w="0.02" h="0.10" d="0.02"/>
         </link>
         <!-- 机器人的关节 用于组合机器人的部件-->

File: chapt6/chapt6_ws/src/fishbot_description/urdf/fishbot/sensor/laser.urdf.xacro (robot description, xacro)
@@ -1,4 +1,5 @@
 <?xml version="1.0"?>
 <robot xmlns:xacro="http://www.ros.org/wiki/xacro">
+    <xacro:include filename="$(find fishbot_description)/urdf/fishbot/common_intertia.urdf.xacro"/>
     <xacro:macro name="laser_xacro" params="xyz">
         <link name="laser_cylinder_link">
@@ -9,5 +10,4 @@
                 <!-- 几何形状 -->
                 <geometry>
-                    <!-- 正方体 -->
                     <cylinder radius="0.01" length="0.10"/>
                 </geometry>
@@ -17,4 +17,17 @@
                 </material>
             </visual>
+            <collision>
+                <!-- 沿着自身几何中心的偏移量和旋转量 -->
+                <origin xyz="0.0 0.0 0.0" rpy="0.0 0.0 0.0"/>
+                <!-- 几何形状 -->
+                <geometry>
+                    <cylinder radius="0.01" length="0.10"/>
+                </geometry>
+                <!-- 材质 颜色 -->
+                <material name="black">
+                    <color rgba="0.0 0.0 0.0 1.0"/>
+                </material>
+            </collision>
+            <xacro:cylinder_intertia m="0.1" r="0.01" h="0.10"/>
         </link>
         <link name="laser_link">
@@ -25,5 +38,4 @@
                 <!-- 几何形状 -->
                 <geometry>
-                    <!-- 正方体 -->
                     <cylinder radius="0.02" length="0.02"/>
                 </geometry>
@@ -33,4 +45,17 @@
                 </material>
             </visual>
+            <collision>
+                <!-- 沿着自身几何中心的偏移量和旋转量 -->
+                <origin xyz="0.0 0.0 0.0" rpy="0.0 0.0 0.0"/>
+                <!-- 几何形状 -->
+                <geometry>
+                    <cylinder radius="0.02" length="0.02"/>
+                </geometry>
+                <!-- 材质 颜色 -->
+                <material name="black">
+                    <color rgba="0.0 0.0 0.0 1.0"/>
+                </material>
+            </collision>
+            <xacro:cylinder_intertia m="0.05" r="0.02" h="0.02"/>
         </link>
         <!-- 机器人的关节 用于组合机器人的部件-->
